File: FF OSD Adapter - Rev 2/FF OSD Adapter - Rev 2.sch (KiCad schematic (older format))
At the start: 10 parts, among them CN1 Conn_01x09, CN2 Conn_01x09, CN3 Conn_01x04, CN4 Conn_01x04, U1 YAAJ_BluePill_Part_Like

Commit message: Added PND and PDF files
Connections:
- no-connect marks 1 -> 21
Changed lines of the file:
@@
 L power:+3.3V #PWR0108
 U 1 1 605F92B2
-P 4775 2475
-F 0 "#PWR0108" H 4775 2325 50  0001 C CNN
-F 1 "+3.3V" V 4790 2603 50  0000 L CNN
-F 2 "" H 4775 2475 50  0001 C CNN
-F 3 "" H 4775 2475 50  0001 C CNN
-	1    4775 2475
+P 4975 2475
+F 0 "#PWR0108" H 4975 2325 50  0001 C CNN
+F 1 "+3.3V" V 4990 2603 50  0000 L CNN
+F 2 "" H 4975 2475 50  0001 C CNN
+F 3 "" H 4975 2475 50  0001 C CNN
+	1    4975 2475
 	0    1    1    0
 $EndComp
 Wire Wire Line
-	4575 2475 4775 2475
+	4575 2475 4975 2475
 $Comp
 L power:+3.3V #PWR0110
@@
 	0    -1   -1   0
 $EndComp
-Wire Wire Line
-	4575 3675 4750 3675
-Wire Wire Line
-	4575 3775 4750 3775
 Text GLabel 4125 6400 0    50   Input ~ 0
 DISPLAY_OUTPUT
@@
 Wire Wire Line
 	4475 6400 4925 6400
-Wire Wire Line
-	4750 3775 4750 3875
-Wire Wire Line
-	4750 3875 4925 3875
-Wire Wire Line
-	4750 3675 4750 3575
-Wire Wire Line
-	4750 3575 4925 3575
 $Comp
 L power:+5V #PWR0102
@@
 Text GLabel 4575 2775 2    50   Input ~ 0
 BT3
+NoConn ~ 4575 3575
+NoConn ~ 2975 2275
+NoConn ~ 2975 2375
+NoConn ~ 2975 2975
+NoConn ~ 2975 3075
+NoConn ~ 2975 3475
+NoConn ~ 2975 4175
+NoConn ~ 4575 4175
+NoConn ~ 4575 4075
+NoConn ~ 4575 3975
+NoConn ~ 4575 3875
+NoConn ~ 4575 3475
+NoConn ~ 4575 3375
+NoConn ~ 4575 3275
+NoConn ~ 4575 3175
+NoConn ~ 4575 3075
+NoConn ~ 4575 2975
+NoConn ~ 4575 2875
+NoConn ~ 4575 2675
+NoConn ~ 4575 2575
+Text GLabel 4575 3775 2    50   Input ~ 0
+A0
+Text GLabel 4575 3675 2    50   Input ~ 0
+A1
+$Comp
+L power:PWR_FLAG #FLG0102
+U 1 1 60A15DA4
+P 2425 4075
+F 0 "#FLG0102" H 2425 4150 50  0001 C CNN
+F 1 "PWR_FLAG" V 2425 4202 50  0000 L CNN
+F 2 "" H 2425 4075 50  0001 C CNN
+F 3 "~" H 2425 4075 50  0001 C CNN
+	1    2425 4075
+	0    -1   -1   0
+$EndComp
+Connection ~ 2425 4075
+$Comp
+L power:PWR_FLAG #FLG0103
+U 1 1 60A15F56
+P 4975 2475
+F 0 "#FLG0103" H 4975 2550 50  0001 C CNN
+F 1 "PWR_FLAG" V 4975 2602 50  0000 L CNN
+F 2 "" H 4975 2475 50  0001 C CNN
+F 3 "~" H 4975 2475 50  0001 C CNN
+	1    4975 2475
+	-1   0    0    1
+$EndComp
+Connection ~ 4975 2475
 Text GLabel 4575 3575 2    50   Input ~ 0
 A2
-NoConn ~ 4575 3575
+Text GLabel 5250 3500 2    50   Input ~ 0
+A2
+NoConn ~ 5250 3500
 $EndSCHEMATC
